Commit message: refactor for connecting to other link

File: ur_description/urdf/inc/ur_macro.xacro (robot description, xacro)
@@ -41,4 +41,6 @@
      - Ajit Krisshna N L
      - Muhammad Asif Rana
+    Refactor by WHI for connecting to other link
+     - Xinjue Zou
   -->
   <xacro:include filename="$(find ur_description)/urdf/inc/ur_transmissions.xacro" />
@@ -53,5 +55,6 @@
     safety_limits:=false
     safety_pos_margin:=0.15
-    safety_k_position:=20"
+    safety_k_position:=20
+    connected_to:='' connected_xyz=:'0 0 0' connected_rpy=:'0 0 0'"
   >
     <!-- Load configuration data from the provided .yaml files -->
@@ -63,4 +66,11 @@
     <!-- Add URDF transmission elements (for ros_control) -->
     <xacro:ur_arm_transmission prefix="${prefix}" hw_interface="${transmission_hw_interface}" />
+    <xacro:unless value="${not connected_to}">
+      <joint name="${prefix}joint_${connected_to}" type="fixed">
+        <origin xyz="${connected_xyz}" rpy="${connected_rpy}"/>
+        <parent link="${connected_to}"/>
+        <child link="${prefix}base_link"/>
+      </joint>
+    </xacro:unless>
     <!-- links: main serial chain -->
     <link name="${prefix}base_link"/>

File: ur_description/urdf/ur.xacro (robot description, xacro)
@@ -1,4 +1,9 @@
+<!--
+    Refactor by WHI for connecting to other link
+     - Xinjue Zou
+-->
 <?xml version="1.0"?>
-<robot xmlns:xacro="http://wiki.ros.org/xacro" name="$(arg robot_model)_robot">
+<!-- <robot xmlns:xacro="http://wiki.ros.org/xacro" name="$(arg robot_model)_robot"> -->
+<robot xmlns:xacro="http://wiki.ros.org/xacro" name="ur_robot">
    <!-- import main macro -->
    <xacro:include filename="$(find ur_description)/urdf/inc/ur_macro.xacro"/>
@@ -17,7 +22,11 @@
    <xacro:arg name="safety_pos_margin" default="0.15"/>
    <xacro:arg name="safety_k_position" default="20"/>
+   <xacro:arg name="prefix" default=""/>
+   <xacro:arg name="connected_to" default=""/>
+   <xacro:arg name="connected_xyz" default="0 0 0"/>
+   <xacro:arg name="connected_to" default="0 0 0"/>
    <!-- arm -->
    <xacro:ur_robot
-     prefix=""
+     prefix="$(arg prefix)"
      joint_limits_parameters_file="$(arg joint_limit_params)"
      kinematics_parameters_file="$(arg kinematics_params)"
@@ -27,4 +36,8 @@
      safety_limits="$(arg safety_limits)"
      safety_pos_margin="$(arg safety_pos_margin)"
-     safety_k_position="$(arg safety_k_position)"/>
+     safety_k_position="$(arg safety_k_position)"
+     connected_to="$(arg connected_to)"
+     connected_xyz="$(arg connected_xyz)"
+     connected_rpy="$(arg connected_rpy)"
+     />
 </robot>
